Commit message: Adding new distal meshes

File: sr_description/hand/xacro/finger/distal/distal.urdf.xacro (robot description, xacro)
@@ -53,5 +53,5 @@
 		<xacro:unless value="${bt_sp}">
                   <!-- Standard distal  -->
-                  <mesh filename="package://sr_description/meshes/hand/F1.dae"
+                  <mesh filename="package://sr_description/meshes/hand/F1_new1.stl"
 			scale="0.001 0.001 0.001" />
 		</xacro:unless>

File: sr_description/hand/xacro/thumb/thdistal.urdf.xacro (robot description, xacro)
@@ -147,5 +147,5 @@
 		<xacro:unless value="${bt_sp}">
 		  <!-- Standard distal  -->
-                  <mesh filename="package://sr_description/meshes/hand/TH1_z.dae"
+                  <mesh filename="package://sr_description/meshes/hand/TH1_z_new1.stl"
 			scale="0.001 0.001 0.001" />
 		</xacro:unless>
