Commit message: Names and versions refactores. Missing robots and tests

File: sr_description/hand/xacro/finger/distal/distal.gazebo.xacro (robot description, xacro)
@@ -2,5 +2,4 @@
 <robot xmlns:xacro="http://www.ros.org/wiki/xacro">
   <xacro:macro name="distal_gazebo" params="prefix:=^ link_prefix:=^ tip_sensor:=^|std ns:=^|''">
-    <!-- prefix can be anything but usually is "r_" or  "l_" for right and left hands distinction -->
     <gazebo reference="${prefix}${link_prefix}distal">
       <xacro:unless value="${'none' in tip_sensor}" >

File: sr_description/hand/xacro/finger/distal/distal.transmission.xacro (robot description, xacro)
@@ -1,10 +1,7 @@
 <?xml version="1.0"?>
-<robot xmlns:sensor="http://playerstage.sourceforge.net/gazebo/xmlschema/#sensor"
+<robot xmlns:xacro="http://www.ros.org/wiki/xacro"
+       xmlns:sensor="http://playerstage.sourceforge.net/gazebo/xmlschema/#sensor"
        xmlns:controller="http://playerstage.sourceforge.net/gazebo/xmlschema/#controller"
-       xmlns:interface="http://playerstage.sourceforge.net/gazebo/xmlschema/#interface"
-       xmlns:xacro="http://www.ros.org/wiki/xacro">
-  <!-- prefix can be anything but usually is "r_" or  "l_" for right and left hands distinction -->
-  <!-- link_prefix prepends fingername to the link names -->
-  <!-- joint_prefix prepends fingername to the joint names -->
+       xmlns:interface="http://playerstage.sourceforge.net/gazebo/xmlschema/#interface">
   <xacro:macro name="distal_transmission" params="hand_type:=^ prefix:=^ joint_prefix:=^ link_prefix:=^" >
    <!-- muscle hand -->

File: sr_description/hand/xacro/finger/distal/distal.urdf.xacro (robot description, xacro)
@@ -1,114 +1,83 @@
 <robot xmlns:xacro="http://www.ros.org/wiki/xacro"
-xmlns:sensor="http://playerstage.sourceforge.net/gazebo/xmlschema/#sensor"
-xmlns:controller="http://playerstage.sourceforge.net/gazebo/xmlschema/#controller"
-xmlns:joint="http://playerstage.sourceforge.net/gazebo/xmlschema/#slider"
-xmlns:interface="http://playerstage.sourceforge.net/gazebo/xmlschema/#interface"
-xmlns:body="http://playerstage.sourceforge.net/gazebo/xmlschema/#body"
-xmlns:geom="http://playerstage.sourceforge.net/gazebo/xmlschema/#geom">
+       xmlns:sensor="http://playerstage.sourceforge.net/gazebo/xmlschema/#sensor"
+       xmlns:controller="http://playerstage.sourceforge.net/gazebo/xmlschema/#controller"
+       xmlns:joint="http://playerstage.sourceforge.net/gazebo/xmlschema/#slider"
+       xmlns:interface="http://playerstage.sourceforge.net/gazebo/xmlschema/#interface"
+       xmlns:body="http://playerstage.sourceforge.net/gazebo/xmlschema/#body"
+       xmlns:geom="http://playerstage.sourceforge.net/gazebo/xmlschema/#geom">
   <xacro:include filename="$(find sr_description)/hand/xacro/finger/distal/distal.gazebo.xacro" />
   <xacro:include filename="$(find sr_description)/hand/xacro/finger/distal/distal.transmission.xacro" />
-  <!-- tip_sensor describes the sensor std, none, bio, bt_sp, ubi, eli -->
-  <!-- prefix can be anything but usually is "r_" or  "l_" for right and left hands distinction -->
-  <!-- link_prefix prepends fingername to the link names -->
-  <!-- joint_prefix prepends fingername to the joint names -->
-  <!-- parent is the parent link for the joint -->
-  <xacro:macro name="distal"
-  params="prefix:=^ link_prefix:=^ joint_prefix:=^ tip_sensor:=^|'std' parent">
+  <xacro:macro name="distal" params="prefix:=^ link_prefix:=^ joint_prefix:=^ tip_sensor:=^|'std' parent">
     <link name="${prefix}${link_prefix}distal">
       <inertial>
         <mass value="0.012" />
         <origin xyz="0 0 0.012" />
-        <inertia ixx="0.00000094" ixy="0.0" ixz="0.0"
-		 iyy="0.0000011" iyz="0.0" izz="0.00000053" />
+        <inertia ixx="0.00000094" ixy="0.0" ixz="0.0" iyy="0.0000011" iyz="0.0" izz="0.00000053" />
       </inertial>
-      <visual>
-        <origin xyz="0 0 0" rpy="0 0 0" />
-        <geometry name="${prefix}${link_prefix}distal_visual">
-          <xacro:unless value="${tip_sensor in ['ubi','bt_sp','eli']}">
-            <!-- Standard distal  -->
-            <mesh filename="package://sr_description/meshes/hand/F1.dae"
+      <xacro:if value="${tip_sensor in ['ubi']}">
+        <visual>
+          <origin xyz="0 0 0" rpy="0 0 0" />
+          <geometry name="${prefix}${link_prefix}distal_visual">
+            <mesh filename="package://sr_description/meshes/components/f_distal/ubi/ubi_tip_visual.dae"
                   scale="0.001 0.001 0.001" />
-          </xacro:unless>
-          <xacro:if value="${tip_sensor in ['ubi','bt_sp','eli']}">
-            <xacro:if value="${'ubi' in tip_sensor}">
-              <!-- Ubi distal -->
-              <mesh filename="package://sr_description/meshes/hand/ubi_tactiles/ubi_tip_visual.dae"
-        scale="0.001 0.001 0.001" />
-            </xacro:if>
-            <xacro:if value="${'eli' in tip_sensor}">
-              <!-- Ellispoid distal  -->
-              <mesh filename="package://sr_description/meshes/hand/ellipsoids/distal_ellipsoid_visual.dae"
-		    scale="0.001 0.001 0.001" />
-            </xacro:if>
-            <xacro:if value="${'bt_sp' in tip_sensor}">
-              <!-- bt_sp distal  -->
-              <mesh filename="package://sr_description/meshes/hand/biotacs/sp.dae" />
-            </xacro:if>
-          </xacro:if>
-        </geometry>
-        <material name="Grey" />
-      </visual>
-      <collision>
-        <origin xyz="0 0 0" rpy="0 0 0" />
-        <geometry name="${prefix}${link_prefix}distal_collision_geom">
-          <xacro:if value="${tip_sensor in ['ubi','bt_sp','eli']}">
-            <xacro:if value="${'ubi' in tip_sensor}">
-              <!-- Ubi distal -->
-              <mesh filename="package://sr_description/meshes/hand/ubi_tactiles/ubi_tip_collision.dae"
-                    scale="0.001 0.001 0.001" />
-            </xacro:if>
-            <xacro:if value="${'eli' in tip_sensor}">
-              <!-- Ellispoid distal  -->
-              <mesh filename="package://sr_description/meshes/hand/ellipsoids/distal_ellipsoid.dae"
-                    scale="0.001 0.001 0.001" />
-            </xacro:if>
-            <xacro:if value="${'bt_sp' in tip_sensor}">
-              <!-- bt_sp distal  -->
-              <mesh filename="package://sr_description/meshes/hand/biotacs/sp.dae" />
-            </xacro:if>
-          </xacro:if>
-          <xacro:unless value="${tip_sensor in ['ubi','bt_sp','eli']}">
-            <!-- Standard distal  -->
-            <mesh filename="package://sr_description/meshes/hand/F1.dae"
+          </geometry>
+          <material name="Grey" />
+        </visual>
+        <collision>
+          <origin xyz="0 0 0" rpy="0 0 0" />
+          <geometry name="${prefix}${link_prefix}distal_collision_geom">
+            <mesh filename="package://sr_description/meshes/components/f_distal/ubi/ubi_tip_collision.dae"
                   scale="0.001 0.001 0.001" />
-          </xacro:unless>
-        </geometry>
-      </collision>
+          </geometry>
+        </collision>
+      </xacro:if>
+      <xacro:unless value="${tip_sensor in ['ubi']}">
+        <visual>
+          <origin xyz="0 0 0" rpy="0 0 0" />
+          <geometry name="${prefix}${link_prefix}distal_visual">
+            <mesh filename="package://sr_description/meshes/components/f_distal/${tip_sensor}/f_distal_${tip_sensor}.stl"
+                  scale="0.001 0.001 0.001" />
+          </geometry>
+          <material name="Grey" />
+        </visual>
+        <collision>
+          <origin xyz="0 0 0" rpy="0 0 0" />
+          <geometry name="${prefix}${link_prefix}distal_collision_geom">
+            <mesh filename="package://sr_description/meshes/components/f_distal/${tip_sensor}/f_distal_${tip_sensor}.stl"
+                  scale="0.001 0.001 0.001" />
+          </geometry>
+        </collision>
+      </xacro:unless>
     </link>
-    <xacro:unless value="${'bio' in tip_sensor}">
-      <joint name="${prefix}${joint_prefix}J1" type="revolute">
-        <parent link="${parent}" />
-        <child link="${prefix}${link_prefix}distal" />
-        <origin xyz="0 0 0.025" rpy="0 0 0" />
-        <axis xyz="1 0 0" />
-        <xacro:if value="${bio}">
-          <!-- biotac fixed distal joint -->
-          <limit lower="${20/180*pi}" upper="${20/180*pi}"
-          effort="10" velocity="2.0" />
-        </xacro:if>
-        <xacro:unless value="${bio}">
-          <!-- standard distal joint -->
-          <limit lower="0" upper="${pi/2}" effort="2"
-          velocity="2.0" />
-        </xacro:unless>
-        <dynamics damping="0.1" />
-      </joint>
-      <gazebo reference="${prefix}${joint_prefix}J1">
-        <provideFeedback>1</provideFeedback>
-        <implicitSpringDamper>1</implicitSpringDamper>
-      </gazebo>
-      <link name="${prefix}${link_prefix}tip">
-        <inertial>
-          <mass value="0.001" />
-          <inertia ixx="0.0" ixy="0.0" ixz="0.0" iyy="0.0"
-          iyz="0.0" izz="0.0" />
-        </inertial>
-      </link>
-      <joint name="${prefix}${joint_prefix}tip" type="fixed">
-        <parent link="${prefix}${link_prefix}distal" />
-        <child link="${prefix}${link_prefix}tip" />
-        <origin xyz="0 0 0.026" rpy="0 0 0" />
-      </joint>
-    </xacro:unless>
+    <joint name="${prefix}${joint_prefix}J1" type="revolute">
+      <parent link="${parent}" />
+      <child link="${prefix}${link_prefix}distal" />
+      <origin xyz="0 0 0.025" rpy="0 0 0" />
+      <axis xyz="1 0 0" />
+      <xacro:if value="${'bt_2p' in tip_sensor}">
+        <!-- bt_2p fixed distal joint -->
+        <limit lower="${20/180*pi}" upper="${20/180*pi}" effort="10" velocity="2.0" />
+      </xacro:if>
+      <xacro:unless value="${'bt_2p' in tip_sensor}">
+        <!-- standard distal joint -->
+        <limit lower="0" upper="${pi/2}" effort="2" velocity="2.0" />
+      </xacro:unless>
+      <dynamics damping="0.1" />
+    </joint>
+    <gazebo reference="${prefix}${joint_prefix}J1">
+      <provideFeedback>1</provideFeedback>
+      <implicitSpringDamper>1</implicitSpringDamper>
+    </gazebo>
+    <link name="${prefix}${link_prefix}tip">
+      <inertial>
+        <mass value="0.001" />
+        <inertia ixx="0.0" ixy="0.0" ixz="0.0" iyy="0.0" iyz="0.0" izz="0.0" />
+      </inertial>
+    </link>
+    <joint name="${prefix}${joint_prefix}tip" type="fixed">
+      <parent link="${prefix}${link_prefix}distal" />
+      <child link="${prefix}${link_prefix}tip" />
+      <origin xyz="0 0 0.026" rpy="0 0 0" />
+    </joint>
     <!-- extensions -->
     <xacro:distal_gazebo />

File: sr_description/hand/xacro/finger/fingers.urdf.xacro (robot description, xacro)
@@ -5,21 +5,17 @@
   <xacro:include filename="$(find sr_description)/hand/xacro/finger/distal/distal.urdf.xacro" />
   <xacro:include filename="$(find sr_description)/hand/xacro/finger/lfmetacarpal/lfmetacarpal.urdf.xacro" />
-  <xacro:include filename="$(find sr_description)/hand/xacro/finger/biotac/biotac.urdf.xacro" />
-  <!-- lf is true for little finger or false for standard finger -->
-  <!-- tip_sensor describes the sensor none, bio, bt_sp, ubi, eli -->
-  <!-- mid_sensor describes the sensor none, bio, ubi -->
-  <!-- prox_sensor describes the sensor none, standard, ubi -->
-  <!-- reflect is either 1 (for right hand) or -1 (for left hand) -->
-  <!-- prefix can be anything but usually is "r_" or  "l_" for right and left hands distinction -->
+  <xacro:include filename="$(find sr_description)/hand/xacro/finger/middle/middle_and_distal_bt_2p.urdf.xacro" />
   <!-- link_prefix prepends fingername to the link names -->
   <!-- joint_prefix prepends fingername to the joint names -->
   <!-- parent is the parent link for the first joint -->
   <xacro:macro name="finger"
-  params="tip_sensor:=^|'std' mid_sensor:=^|'std' prox_sensor:=^|'std' reflect:=^ prefix:=^ link_prefix joint_prefix parent *origin *axis">
+               params="hand_type:=^ hand_version:=^
+                       tip_sensor:=^|'std' mid_sensor:=^|'std' prox_sensor:=^|'std'
+                       reflect:=^ prefix:=^ link_prefix joint_prefix parent *origin *axis">
     <!-- Little finger special case -->
     <xacro:if value="${'lf' in link_prefix}">
       <xacro:lfmetacarpal parent="${parent}" />
       <!-- Knuckle -->
-      <xacro:knuckle parent="${prefix}lfmetacarpal">
+      <xacro:knuckle hand_type="${hand_type}" hand_version="${hand_version}" parent="${prefix}lfmetacarpal">
         <xacro:insert_block name="origin" />
       </xacro:knuckle>
@@ -28,23 +24,22 @@
     <xacro:unless value="${'lf' in link_prefix}">
       <!-- Knuckle -->
-      <xacro:knuckle parent="${parent}">
+      <xacro:knuckle hand_type="${hand_type}" hand_version="${hand_version}" parent="${parent}">
         <xacro:insert_block name="origin" />
       </xacro:knuckle>
     </xacro:unless>
     <!-- Proximal -->
-    <xacro:proximal parent="${prefix}${link_prefix}knuckle"></xacro:proximal>
+    <xacro:proximal hand_type="${hand_type}" hand_version="${hand_version}" parent="${prefix}${link_prefix}knuckle"/>
     <!-- Biotac Middle -->
-    <xacro:if value="${'bio' in tip_sensor}">
-      <xacro:biotac_middle parent="${prefix}${link_prefix}proximal">
-      </xacro:biotac_middle>
+    <xacro:if value="${'bt_2p' in tip_sensor}">
+      <xacro:middle_and_distal_bt_2p hand_type="${hand_type}" hand_version="${hand_version}" parent="${prefix}${link_prefix}proximal"/>
     </xacro:if>
     <!-- Standard Middle -->
-    <xacro:unless value="${'bio' in tip_sensor}">
-      <xacro:middle parent="${prefix}${link_prefix}proximal"></xacro:middle>
+    <xacro:unless value="${'bt_2p' in tip_sensor}">
+      <xacro:middle hand_type="${hand_type}" hand_version="${hand_version}" parent="${prefix}${link_prefix}proximal"/>
     </xacro:unless>
     <!-- Distal  -->
     <!-- only if finger is not biotac  -->
-    <xacro:unless value="${'bio' in tip_sensor}">
-      <xacro:distal parent="${prefix}${link_prefix}middle"></xacro:distal>
+    <xacro:unless value="${'bt_2p' in tip_sensor}">
+      <xacro:distal parent="${prefix}${link_prefix}middle"/>
     </xacro:unless>
   </xacro:macro>

File: sr_description/hand/xacro/finger/knuckle/knuckle.gazebo.xacro (robot description, xacro)
@@ -2,5 +2,4 @@
 <robot xmlns:xacro="http://www.ros.org/wiki/xacro">
   <xacro:macro name="knuckle_gazebo" params="prefix:=^ link_prefix:=^">
-    <!-- prefix can be anything but usually is "r_" or  "l_" for right and left hands distinction -->
     <gazebo reference="${prefix}${link_prefix}knuckle">
     <!-- knuckle is not highly exposed so bumper seems not useful

File: sr_description/hand/xacro/finger/knuckle/knuckle.transmission.xacro (robot description, xacro)
@@ -1,10 +1,7 @@
 <?xml version="1.0"?>
-<robot xmlns:sensor="http://playerstage.sourceforge.net/gazebo/xmlschema/#sensor"
+<robot xmlns:xacro="http://www.ros.org/wiki/xacro"
+       xmlns:sensor="http://playerstage.sourceforge.net/gazebo/xmlschema/#sensor"
        xmlns:controller="http://playerstage.sourceforge.net/gazebo/xmlschema/#controller"
-       xmlns:interface="http://playerstage.sourceforge.net/gazebo/xmlschema/#interface"
-       xmlns:xacro="http://www.ros.org/wiki/xacro">
-    <!-- prefix can be anything but usually is "r_" or  "l_" for right and left hands distinction -->
-    <!-- link_prefix prepends fingername to the link names -->
-    <!-- joint_prefix prepends fingername to the joint names -->
+       xmlns:interface="http://playerstage.sourceforge.net/gazebo/xmlschema/#interface">
     <xacro:macro name="knuckle_transmission" params="hand_type:=^ prefix:=^ joint_prefix:=^ link_prefix:=^">
         <!-- muscle hand -->

File: sr_description/hand/xacro/finger/knuckle/knuckle.urdf.xacro (robot description, xacro)
@@ -1,29 +1,23 @@
 <robot xmlns:xacro="http://www.ros.org/wiki/xacro"
-xmlns:sensor="http://playerstage.sourceforge.net/gazebo/xmlschema/#sensor"
-xmlns:controller="http://playerstage.sourceforge.net/gazebo/xmlschema/#controller"
-xmlns:joint="http://playerstage.sourceforge.net/gazebo/xmlschema/#slider"
-xmlns:interface="http://playerstage.sourceforge.net/gazebo/xmlschema/#interface"
-xmlns:body="http://playerstage.sourceforge.net/gazebo/xmlschema/#body"
-xmlns:geom="http://playerstage.sourceforge.net/gazebo/xmlschema/#geom">
+       xmlns:sensor="http://playerstage.sourceforge.net/gazebo/xmlschema/#sensor"
+       xmlns:controller="http://playerstage.sourceforge.net/gazebo/xmlschema/#controller"
+       xmlns:joint="http://playerstage.sourceforge.net/gazebo/xmlschema/#slider"
+       xmlns:interface="http://playerstage.sourceforge.net/gazebo/xmlschema/#interface"
+       xmlns:body="http://playerstage.sourceforge.net/gazebo/xmlschema/#body"
+       xmlns:geom="http://playerstage.sourceforge.net/gazebo/xmlschema/#geom">
   <xacro:include filename="$(find sr_description)/hand/xacro/finger/knuckle/knuckle.gazebo.xacro" />
   <xacro:include filename="$(find sr_description)/hand/xacro/finger/knuckle/knuckle.transmission.xacro" />
-  <!-- prefix can be anything but usually is "r_" or  "l_" for right and left hands distinction -->
-  <!-- link_prefix prepends fingername to the link names -->
-  <!-- joint_prefix prepends fingername to the joint names -->
-  <!-- parent is the parent link for the joint -->
-  <xacro:macro name="knuckle"
-  params="prefix:=^ link_prefix:=^ joint_prefix:=^ parent *origin">
+  <xacro:macro name="knuckle" params="hand_type:=^ hand_version:=^ prefix:=^ link_prefix:=^ joint_prefix:=^ parent *origin">
     <link name="${prefix}${link_prefix}knuckle">
       <inertial>
         <origin xyz="0 0 0" rpy="0 0 0" />
         <mass value="0.008" />
-        <inertia ixx="0.00000026" ixy="0.0" ixz="0.0"
-        iyy="0.00000026" iyz="0.0" izz="0.00000032" />
+        <inertia ixx="0.00000026" ixy="0.0" ixz="0.0" iyy="0.00000026" iyz="0.0" izz="0.00000032" />
       </inertial>
       <visual>
         <origin xyz="0 0 0.0005" rpy="0 0 0" />
         <geometry name="${prefix}${link_prefix}knuckle_visual">
-          <mesh filename="package://sr_description/meshes/hand/knuckle.dae"
-          scale="0.001 0.001 0.001" />
+          <mesh filename="package://sr_description/meshes/products/${hand_type}/${hand_version}/f_knuckle_${hand_version}.dae"
+                scale="0.001 0.001 0.001" />
         </geometry>
         <material name="LightGrey" />
@@ -39,9 +33,7 @@
       <parent link="${parent}" />
       <child link="${prefix}${link_prefix}knuckle" />
-      <!--<origin xyz="0.033 0 0.095" rpy="0 0 0" />-->
       <xacro:insert_block name="origin" />
       <xacro:insert_block name="axis" />
-      <limit lower="${-20/180*pi}" upper="${20/180*pi}"
-      effort="2" velocity="2.0" />
+      <limit lower="${-20/180*pi}" upper="${20/180*pi}" effort="2" velocity="2.0" />
       <dynamics damping="0.1" />
     </joint>

File: sr_description/hand/xacro/finger/lfmetacarpal/lfmetacarpal.gazebo.xacro (robot description, xacro)
@@ -2,5 +2,4 @@
 <robot xmlns:xacro="http://www.ros.org/wiki/xacro">
   <xacro:macro name="lfmetacarpal_gazebo" params="prefix:=^ palm_sensor:=^|std link_prefix">
-    <!-- prefix can be anything but usually is "r_" or  "l_" for right and left hands distinction -->
     <gazebo reference="${prefix}lfmetacarpal">
       <xacro:unless value="${'none' in palm_sensor}" >

File: sr_description/hand/xacro/finger/lfmetacarpal/lfmetacarpal.transmission.xacro (robot description, xacro)
@@ -1,8 +1,7 @@
 <?xml version="1.0"?>
-<robot xmlns:sensor="http://playerstage.sourceforge.net/gazebo/xmlschema/#sensor"
+<robot xmlns:xacro="http://www.ros.org/wiki/xacro"
+       xmlns:sensor="http://playerstage.sourceforge.net/gazebo/xmlschema/#sensor"
        xmlns:controller="http://playerstage.sourceforge.net/gazebo/xmlschema/#controller"
-       xmlns:interface="http://playerstage.sourceforge.net/gazebo/xmlschema/#interface"
-       xmlns:xacro="http://www.ros.org/wiki/xacro">
-    <!-- prefix can be anything but usually is "r_" or  "l_" for right and left hands distinction -->
+       xmlns:interface="http://playerstage.sourceforge.net/gazebo/xmlschema/#interface">
     <xacro:macro name="lfmetacarpal_transmission" params="hand_type:=^ prefix:=^">
         <!-- muscle hand -->

File: sr_description/hand/xacro/finger/lfmetacarpal/lfmetacarpal.urdf.xacro (robot description, xacro)
@@ -1,14 +1,11 @@
 <robot xmlns:xacro="http://www.ros.org/wiki/xacro"
-xmlns:sensor="http://playerstage.sourceforge.net/gazebo/xmlschema/#sensor"
-xmlns:controller="http://playerstage.sourceforge.net/gazebo/xmlschema/#controller"
-xmlns:joint="http://playerstage.sourceforge.net/gazebo/xmlschema/#slider"
-xmlns:interface="http://playerstage.sourceforge.net/gazebo/xmlschema/#interface"
-xmlns:body="http://playerstage.sourceforge.net/gazebo/xmlschema/#body"
-xmlns:geom="http://playerstage.sourceforge.net/gazebo/xmlschema/#geom">
+       xmlns:sensor="http://playerstage.sourceforge.net/gazebo/xmlschema/#sensor"
+       xmlns:controller="http://playerstage.sourceforge.net/gazebo/xmlschema/#controller"
+       xmlns:joint="http://playerstage.sourceforge.net/gazebo/xmlschema/#slider"
+       xmlns:interface="http://playerstage.sourceforge.net/gazebo/xmlschema/#interface"
+       xmlns:body="http://playerstage.sourceforge.net/gazebo/xmlschema/#body"
+       xmlns:geom="http://playerstage.sourceforge.net/gazebo/xmlschema/#geom">
   <xacro:include filename="$(find sr_description)/hand/xacro/finger/lfmetacarpal/lfmetacarpal.gazebo.xacro" />
   <xacro:include filename="$(find sr_description)/hand/xacro/finger/lfmetacarpal/lfmetacarpal.transmission.xacro" />
-  <!-- prefix can be anything but usually is "r_" or  "l_" for right and left hands distinction -->
-  <!-- reflect is either 1 (for right hand) or -1 (for left hand) -->
-  <!-- parent is the parent link for the joint -->
   <xacro:macro name="lfmetacarpal"
   params="prefix:=^ reflect:=^ parent">
@@ -23,5 +20,5 @@
         <origin xyz="0 0 0" rpy="0 0 0" />
         <geometry name="${prefix}lfmetacarpal_visual">
-          <mesh filename="package://sr_description/meshes/hand/lfmetacarpal.dae"
+          <mesh filename="package://sr_description/meshes/products/${hand_type}/${hand_version}/lf_metacarpal_${hand_version}.dae"
           scale="${reflect*0.001} 0.001 0.001" />
         </geometry>

File: sr_description/hand/xacro/finger/middle/middle.gazebo.xacro (robot description, xacro)
@@ -2,5 +2,4 @@
 <robot xmlns:xacro="http://www.ros.org/wiki/xacro">
   <xacro:macro name="middle_gazebo" params="prefix:=^ link_prefix:=^ mid_sensor:=^|std">
-    <!-- prefix can be anything but usually is "r_" or  "l_" for right and left hands distinction -->
     <gazebo reference="${prefix}${link_prefix}middle">
       <xacro:unless value="${'none' in mid_sensor}">
