Commit message: Names and versions refactores. Missing robots and tests

File: sr_description/hand/xacro/finger/middle/middle.transmission.xacro (robot description, xacro)
@@ -1,10 +1,7 @@
 <?xml version="1.0"?>
-<robot xmlns:sensor="http://playerstage.sourceforge.net/gazebo/xmlschema/#sensor"
+<robot xmlns:xacro="http://www.ros.org/wiki/xacro"
+       xmlns:sensor="http://playerstage.sourceforge.net/gazebo/xmlschema/#sensor"
        xmlns:controller="http://playerstage.sourceforge.net/gazebo/xmlschema/#controller"
-       xmlns:interface="http://playerstage.sourceforge.net/gazebo/xmlschema/#interface"
-       xmlns:xacro="http://www.ros.org/wiki/xacro">
-    <!-- prefix can be anything but usually is "r_" or  "l_" for right and left hands distinction -->
-    <!-- link_prefix prepends fingername to the link names -->
-    <!-- joint_prefix prepends fingername to the joint names -->
+       xmlns:interface="http://playerstage.sourceforge.net/gazebo/xmlschema/#interface">
     <xacro:macro name="middle_transmission" params="hand_type:=^ prefix:=^ joint_prefix:=^ link_prefix:=^">
         <!-- muscle hand -->

File: sr_description/hand/xacro/finger/middle/middle.urdf.xacro (robot description, xacro)
@@ -1,29 +1,23 @@
 <robot xmlns:xacro="http://www.ros.org/wiki/xacro"
-xmlns:sensor="http://playerstage.sourceforge.net/gazebo/xmlschema/#sensor"
-xmlns:controller="http://playerstage.sourceforge.net/gazebo/xmlschema/#controller"
-xmlns:joint="http://playerstage.sourceforge.net/gazebo/xmlschema/#slider"
-xmlns:interface="http://playerstage.sourceforge.net/gazebo/xmlschema/#interface"
-xmlns:body="http://playerstage.sourceforge.net/gazebo/xmlschema/#body"
-xmlns:geom="http://playerstage.sourceforge.net/gazebo/xmlschema/#geom">
+       xmlns:sensor="http://playerstage.sourceforge.net/gazebo/xmlschema/#sensor"
+       xmlns:controller="http://playerstage.sourceforge.net/gazebo/xmlschema/#controller"
+       xmlns:joint="http://playerstage.sourceforge.net/gazebo/xmlschema/#slider"
+       xmlns:interface="http://playerstage.sourceforge.net/gazebo/xmlschema/#interface"
+       xmlns:body="http://playerstage.sourceforge.net/gazebo/xmlschema/#body"
+       xmlns:geom="http://playerstage.sourceforge.net/gazebo/xmlschema/#geom">
   <xacro:include filename="$(find sr_description)/hand/xacro/finger/middle/middle.gazebo.xacro" />
   <xacro:include filename="$(find sr_description)/hand/xacro/finger/middle/middle.transmission.xacro" />
-  <!-- prefix can be anything but usually is "r_" or  "l_" for right and left hands distinction -->
-  <!-- link_prefix prepends fingername to the link names -->
-  <!-- joint_prefix prepends fingername to the joint names -->
-  <!-- parent is the parent link for the joint -->
-  <xacro:macro name="middle"
-  params="prefix:=^ link_prefix:=^ joint_prefix:=^ parent">
+  <xacro:macro name="middle" params="hand_type:=^ hand_version:=^ prefix:=^ link_prefix:=^ joint_prefix:=^ parent">
     <link name="${prefix}${link_prefix}middle">
       <inertial>
         <origin xyz="0 0 0.0125" rpy="0 0 0" />
         <mass value="0.017" />
-        <inertia ixx="0.0000026" ixy="0.0" ixz="0.0"
-        iyy="0.0000027" iyz="0.0" izz="0.00000087" />
+        <inertia ixx="0.0000026" ixy="0.0" ixz="0.0" iyy="0.0000027" iyz="0.0" izz="0.00000087" />
       </inertial>
       <visual>
         <origin xyz="0 0 0" rpy="0 0 0" />
         <geometry name="${prefix}${link_prefix}middle_visual">
-          <mesh filename="package://sr_description/meshes/hand/F2.dae"
-          scale="0.001 0.001 0.001" />
+          <mesh filename="package://sr_description/meshes/products/${hand_type}/${hand_version}/f_middle_${hand_version}.dae"
+                scale="0.001 0.001 0.001" />
         </geometry>
         <material name="Grey" />
@@ -53,6 +47,5 @@
       <origin xyz="0 0 0.045" rpy="0 0 0" />
       <axis xyz="1 0 0" />
-      <limit lower="0" upper="${pi/2}" effort="2"
-      velocity="2.0" />
+      <limit lower="0" upper="${pi/2}" effort="2" velocity="2.0" />
       <dynamics damping="0.1" />
     </joint>

File: sr_description/hand/xacro/finger/proximal/proximal.gazebo.xacro (robot description, xacro)
@@ -2,5 +2,4 @@
 <robot xmlns:xacro="http://www.ros.org/wiki/xacro">
   <xacro:macro name="proximal_gazebo" params="prefix:=^ link_prefix:=^ prox_sensor:=^|std">
-    <!-- prefix can be anything but usually is "r_" or  "l_" for right and left hands distinction -->
     <gazebo reference="${prefix}${link_prefix}proximal">
       <xacro:unless value="${'none' in prox_sensor}" >

File: sr_description/hand/xacro/finger/proximal/proximal.transmission.xacro (robot description, xacro)
@@ -4,7 +4,4 @@
        xmlns:interface="http://playerstage.sourceforge.net/gazebo/xmlschema/#interface"
        xmlns:xacro="http://www.ros.org/wiki/xacro">
-    <!-- prefix can be anything but usually is "r_" or  "l_" for right and left hands distinction -->
-    <!-- link_prefix prepends fingername to the link names -->
-    <!-- joint_prefix prepends fingername to the joint names -->
     <xacro:macro name="proximal_transmission" params="hand_type:=^ prefix:=^ joint_prefix:=^ link_prefix:=^">
         <!-- muscle hand -->

File: sr_description/hand/xacro/finger/proximal/proximal.urdf.xacro (robot description, xacro)
@@ -8,22 +8,17 @@
   <xacro:include filename="$(find sr_description)/hand/xacro/finger/proximal/proximal.gazebo.xacro" />
   <xacro:include filename="$(find sr_description)/hand/xacro/finger/proximal/proximal.transmission.xacro" />
-  <!-- prefix can be anything but usually is "r_" or  "l_" for right and left hands distinction -->
-  <!-- link_prefix prepends fingername to the link names -->
-  <!-- joint_prefix prepends fingername to the joint names -->
-  <!-- parent is the parent link for the joint -->
   <xacro:macro name="proximal"
-  params="prefix:=^ link_prefix:=^ joint_prefix:=^ parent">
+               params="hand_type:=^ hand_version:=^ prefix:=^ link_prefix:=^ joint_prefix:=^ parent">
     <link name="${prefix}${link_prefix}proximal">
       <inertial>
         <mass value="0.030" />
         <origin xyz="0 0 0.0225" />
-        <inertia ixx="0.0000098" ixy="0.0" ixz="0.0" iyy="0.00001"
-        iyz="0.0" izz="0.0000018" />
+        <inertia ixx="0.0000098" ixy="0.0" ixz="0.0" iyy="0.00001" iyz="0.0" izz="0.0000018" />
       </inertial>
       <visual>
         <origin xyz="0 0 0" rpy="0 0 0" />
         <geometry name="${prefix}${link_prefix}proximal_visual">
-          <mesh filename="package://sr_description/meshes/hand/F3.dae"
-          scale="0.001 0.001 0.001" />
+          <mesh filename="package://sr_description/meshes/products/${hand_type}/${hand_version}/f_proximal_${hand_version}.dae"
+                scale="0.001 0.001 0.001" />
         </geometry>
         <material name="Grey" />
@@ -41,6 +36,5 @@
       <origin xyz="0 0 0" rpy="0 0 0" />
       <axis xyz="1 0 0" />
-      <limit lower="-${15.0*pi/180}" upper="${pi/2}" effort="2"
-      velocity="2.0" />
+      <limit lower="-${15.0*pi/180}" upper="${pi/2}" effort="2" velocity="2.0" />
       <dynamics damping="0.1" />
     </joint>

File: sr_description/hand/xacro/full_hand.urdf.xacro (robot description, xacro)
@@ -3,10 +3,10 @@
 xmlns:interface="http://playerstage.sourceforge.net/gazebo/xmlschema/#interface"
 xmlns:xacro="http://www.ros.org/wiki/xacro">
-  <xacro:include filename="$(find sr_description)/hand/xacro/forearm/forearm.urdf.xacro" />
+  <xacro:include filename="$(find sr_description)/hand/xacro/forearm/forearm_e.urdf.xacro" />
   <xacro:include filename="$(find sr_description)/hand/xacro/wrist/wrist.urdf.xacro" />
-  <xacro:include filename="$(find sr_description)/hand/xacro/palm/palm.urdf.xacro" />
+  <xacro:include filename="$(find sr_description)/hand/xacro/palm/palm_e.urdf.xacro" />
   <xacro:include filename="$(find sr_description)/hand/xacro/finger/fingers.urdf.xacro" />
   <xacro:include filename="$(find sr_description)/hand/xacro/thumb/thumb.urdf.xacro" />
-  <!-- hand_type describes the hand type, hand_e, hand_e_plus, hand_m (muscle) -->
+  <!-- hand_type describes the hand type, hand_m (muscle), hand_e, hand_g -->
   <!-- fingers describes which fingers are present, [th, ff, mf, rf, lf], default [1, 1, 1, 1, 1] -->
   <!-- muscletrans (deprecated) is true for muscle transmission to be used, false to use motor transmission -->
@@ -21,11 +21,11 @@
   <!-- palm_sensor describes the sensor std, none, ubi -->
   <!-- reflect is either 1 (for right hand) or -1 (for left hand) -->
-  <!-- prefix can be anything but usually is "r_" or  "l_" for right and left hands distinction -->
   <!-- lf (deprecated) is true if we want a little finger, false otherwise -->
   <xacro:macro name="shadowhand"
-  params="hand_type:='hand_e' reflect prefix cable_mesh:=False
-          fingers:=${[1,1,1,1,1]} tip_sensors:=${['std','std','std','std','std']} prox_sensors:=${['std','std','std','std','std']}
-          mid_sensors:=${['std','std','std','std','std']} palm_sensor:=std
-          muscletrans:=False muscle:=False lf:=True bio:=False bt_sp:=False ubi:=False eli:=False">
+               params="hand_type:='hand_e' hand_version:='E3' reflect prefix cable_mesh:=False
+                      fingers:=${[1,1,1,1,1]} tip_sensors:=${['std','std','std','std','std']}
+                      prox_sensors:=${['std','std','std','std','std']}
+                      mid_sensors:=${['std','std','std','std','std']} palm_sensor:=std
+                      muscletrans:=False muscle:=False lf:=True bio:=False bt_sp:=False ubi:=False eli:=False">
     <!-- handle deprecated parameters -->
     <xacro:include filename="$(find sr_description)/hand/xacro/backward_compat.urdf.xacro" />

File: sr_description/hand/xacro/palm/palm.gazebo.xacro (robot description, xacro)
@@ -2,5 +2,4 @@
 <robot xmlns:xacro="http://www.ros.org/wiki/xacro">
   <xacro:macro name="shadowhand_palm_gazebo" params="prefix:=^ palm_sensor:=^|std">
-    <!-- prefix can be anything but usually is "r_" or  "l_" for right and left hands distinction -->
     <gazebo reference="${prefix}palm">
       <xacro:unless value="${'none' in palm_sensor}" >

File: sr_description/hand/xacro/palm/palm.transmission.xacro (robot description, xacro)
@@ -1,8 +1,7 @@
 <?xml version="1.0"?>
-<robot xmlns:sensor="http://playerstage.sourceforge.net/gazebo/xmlschema/#sensor"
+<robot xmlns:xacro="http://www.ros.org/wiki/xacro"
+       xmlns:sensor="http://playerstage.sourceforge.net/gazebo/xmlschema/#sensor"
        xmlns:controller="http://playerstage.sourceforge.net/gazebo/xmlschema/#controller"
-       xmlns:interface="http://playerstage.sourceforge.net/gazebo/xmlschema/#interface"
-       xmlns:xacro="http://www.ros.org/wiki/xacro">
-    <!-- prefix can be anything but usually is "r_" or  "l_" for right and left hands distinction -->
+       xmlns:interface="http://playerstage.sourceforge.net/gazebo/xmlschema/#interface">
     <xacro:macro name="shadowhand_palm_transmission" params="hand_type:=^ prefix:=^">
         <!-- muscle hand -->

File: sr_description/hand/xacro/thumb/thbase.gazebo.xacro (robot description, xacro)
@@ -2,5 +2,4 @@
 <robot xmlns:xacro="http://www.ros.org/wiki/xacro">
   <xacro:macro name="thbase_gazebo" params="prefix:=^">
-    <!-- prefix can be anything but usually is "r_" or  "l_" for right and left hands distinction -->
     <gazebo reference="${prefix}thbase">
       <!-- base is inside the proximal and not exposed so bumper seems useless
