Commit message: Adding mesh of the hand and test it in the palm

File: sr_description/hand/xacro/palm/palm.urdf.xacro (robot description, xacro)
@@ -25,5 +25,5 @@
         <origin xyz="0 0 0" rpy="0 0 0" />
         <geometry name="${prefix}palm_visual">
-          <mesh filename="package://sr_description/meshes/hand/palm.dae"
+          <mesh filename="package://sr_description/meshes/hand/hand.stl"
           scale="${reflect*0.001} 0.001 0.001" />
         </geometry>
