Commit message: Modify the dae and xacro

File: sr_description/arm/xacro/mounting_plate/shadowarm_mounting_plate.urdf.xacro (robot description, xacro)
@@ -3,5 +3,5 @@
     <link name="shadowarm_mounting_plate">
       <visual>
-        <origin xyz="0.0 0.0 -0.01" rpy="0 1.571 0" />
+        <origin xyz="0.0 0.0 0.0" rpy="0 0 0" />
         <geometry name="shadowarm_mounting_plate_visual">
           <mesh filename="package://sr_description/arm/model/mounting_plate.dae"
@@ -11,5 +11,5 @@
       </visual>
       <collision>
-        <origin xyz="0.0 0.0 -0.01" rpy="0 1.571 0" />
+        <origin xyz="0.0 0.0 0.0" rpy="0 0 0" />
         <geometry name="shadowarm_mounting_plate_collision">
           <cylinder length="0.0115" radius="0.074" />
@@ -20,14 +20,4 @@
       <selfCollide>false</selfCollide>
     </gazebo>
-    <joint name="ra_arm_to_mounting_plate" type="fixed">
-      <parent link="ra_ee_link" />
-      <child link="shadowarm_mounting_plate" />
-      <origin xyz="-0.001 0.0 0.0" rpy="${pi/2.0} ${0.0} ${pi/2.0}" />
-    </joint>
-    <joint name="ra_mounting_plate_to_hand" type="fixed">
-      <parent link="shadowarm_mounting_plate" />
-      <child link="rh_forearm" />
-      <origin xyz="0.0 0.0 0.0" rpy="0 0 0" />
-    </joint>
   </xacro:macro>
 </robot>
