Commit message: Fixing inacuracies

File: sr_description/hand/xacro/hand_e.urdf.xacro (robot description, xacro)
@@ -25,5 +25,5 @@
     <!-- Wrist -->
     <xacro:wrist parent="${prefix}forearm">
-      <origin xyz="0 -0.010 0.213" rpy="0 0 0" />
+      <origin xyz="0 -0.010 0.21301" rpy="0 0 0" />
     </xacro:wrist>
     <!-- Palm -->

File: sr_description/hand/xacro/hand_g.urdf.xacro (robot description, xacro)
@@ -28,5 +28,5 @@
       <parent link="${prefix}forearm" />
       <child link="${prefix}palm" />
-      <origin xyz="0 -0.015 0.149" rpy="-${40*pi/180} 0 0" />
+      <origin xyz="0 -0.01569 0.14895" rpy="-${40*pi/180} 0 0" />
       <axis xyz="0 ${reflect} 0" />
     </joint>

File: sr_description/hand/xacro/thumb/thbase.urdf.xacro (robot description, xacro)
@@ -35,5 +35,5 @@
       <parent link="${parent}" />
       <child link="${prefix}thbase" />
-      <origin xyz="${reflect*0.034} -0.0085 0.029"
+      <origin xyz="${reflect*0.034} -0.00858 0.029"
       rpy="0 ${pi/4} ${pi/2-reflect*pi/2}" />
       <axis xyz="0 0 ${reflect*-1}" />
