Commit message: Fix backward compatibility
- Restore deleted files required by compatibility test
- Fix use of deprecated properties
- Fix use of deprecated parameters
- Undo unrelated changes w.r.t. upstream
- Fix extra_lite hands: it is missing MF not FF

File: sr_description/hand/xacro/backward_compat.urdf.xacro (robot description, xacro)
@@ -1,42 +1,35 @@
 <robot xmlns:xacro="http://www.ros.org/wiki/xacro">
   <!-- for backward compatibility define new params from old ones -->
-  <xacro:property name="old_tip_sensor" value="${(1 if bio==True else 0) + (1 if bt_sp==True else 0) + (1 if ubi==True else 0) + (1 if eli==True else 0)}"/>
-  <!-- if old parameters are used, valid only if sum is 1 -->
-  <xacro:if value="${old_tip_sensor==1}">
-    <xacro:if value="${bio}">
-      <xacro:property name="palm_sensor" value="std"/>
-      <xacro:property name="prox_sensor" value="${[std, std, std, std ,std]}"/>
-      <xacro:property name="mid_sensor" value="${[bio, bio, bio, bio ,bio]}"/>
-      <xacro:property name="tip_sensor" value="${[bio, bio, bio, bio ,bio]}"/>
-    </xacro:if>
-    <xacro:if value="${bt_sp}">
-      <xacro:property name="palm_sensor" value="std"/>
-      <xacro:property name="prox_sensor" value="${[std, std, std, std ,std]}"/>
-      <xacro:property name="mid_sensor" value="${[std, std, std, std ,std]}"/>
-      <xacro:property name="tip_sensor" value="${[bt_sp, bt_sp, bt_sp, bt_sp ,bt_sp]}"/>
-    </xacro:if>
-    <xacro:if value="${ubi}">
-      <xacro:property name="palm_sensor" value="ubi_fabric"/>
-      <xacro:property name="prox_sensor" value="${[ubi, ubi, ubi, ubi ,ubi]}"/>
-      <xacro:property name="mid_sensor" value="${[ubi, ubi, ubi, ubi ,ubi]}"/>
-      <xacro:property name="tip_sensor" value="${[ubi, ubi, ubi, ubi ,ubi]}"/>
-    </xacro:if>
-    <xacro:if value="${eli}">
-      <xacro:property name="palm_sensor" value="std"/>
-      <xacro:property name="prox_sensor" value="${[std, std, std, std ,std]}"/>
-      <xacro:property name="mid_sensor" value="${[std, std, std, std ,std]}"/>
-      <xacro:property name="tip_sensor" value="${[eli, eli, eli, eli ,eli]}"/>
-    </xacro:if>
+  <xacro:if value="${bio}">
+    <xacro:property name="palm_sensor" value="std" />
+    <xacro:property name="prox_sensors" value="${['std', 'std', 'std', 'std', 'std']}" />
+    <xacro:property name="mid_sensors" value="${['bio', 'bio', 'bio', 'bio', 'bio']}" />
+    <xacro:property name="tip_sensors" value="${['bio', 'bio', 'bio', 'bio', 'bio']}" />
+  </xacro:if>
+  <xacro:if value="${bt_sp}">
+    <xacro:property name="palm_sensor" value="std" />
+    <xacro:property name="prox_sensors" value="${['std', 'std', 'std', 'std', 'std']}" />
+    <xacro:property name="mid_sensors" value="${['std', 'std', 'std', 'std', 'std']}" />
+    <xacro:property name="tip_sensors" value="${['bt_sp', 'bt_sp', 'bt_sp', 'bt_sp', 'bt_sp']}" />
+  </xacro:if>
+  <xacro:if value="${ubi}">
+    <xacro:property name="palm_sensor" value="ubi_fabric" />
+    <xacro:property name="prox_sensors" value="${['ubi', 'ubi', 'ubi', 'ubi', 'ubi']}" />
+    <xacro:property name="mid_sensors" value="${['ubi', 'ubi', 'ubi', 'ubi', 'ubi']}" />
+    <xacro:property name="tip_sensors" value="${['ubi', 'ubi', 'ubi', 'ubi', 'ubi']}" />
+  </xacro:if>
+  <xacro:if value="${eli}">
+    <xacro:property name="palm_sensor" value="std" />
+    <xacro:property name="prox_sensors" value="${['std', 'std', 'std', 'std', 'std']}" />
+    <xacro:property name="mid_sensors" value="${['std', 'std', 'std', 'std', 'std']}" />
+    <xacro:property name="tip_sensors" value="${['eli', 'eli', 'eli', 'eli', 'eli']}" />
   </xacro:if>
   <xacro:if value="${muscle}">
     <xacro:if value="${muscletrans}">
-      <xacro:property name="hand_type" value="hand_mt"/>
+      <xacro:property name="hand_type" value="hand_mt" />
     </xacro:if>
     <xacro:unless value="${muscletrans}">
-      <xacro:property name="hand_type" value="hand_m"/>
+      <xacro:property name="hand_type" value="hand_m" />
     </xacro:unless>
   </xacro:if>
-  <xacro:unless value="${lf}">
-    <xacro:property name="fingers" value="${[1,1,1,1,0]}"/>
-  </xacro:unless>
 </robot>

File: sr_description/hand/xacro/finger/distal/distal.urdf.xacro (robot description, xacro)
@@ -47,5 +47,5 @@
           </xacro:if>
         </geometry>
-        <material name="Grey" />
+        <!-- <material name="Grey" /> -->
       </visual>
       <collision>
@@ -82,14 +82,7 @@
         <origin xyz="0 0 0.025" rpy="0 0 0" />
         <axis xyz="1 0 0" />
-        <xacro:if value="${bio}">
-          <!-- biotac fixed distal joint -->
-          <limit lower="${20/180*pi}" upper="${20/180*pi}"
-          effort="10" velocity="2.0" />
-        </xacro:if>
-        <xacro:unless value="${bio}">
-          <!-- standard distal joint -->
-          <limit lower="0" upper="${pi/2}" effort="2"
-          velocity="2.0" />
-        </xacro:unless>
+        <!-- standard distal joint -->
+        <limit lower="0" upper="${pi/2}" effort="2"
+        velocity="2.0" />
         <dynamics damping="0.1" />
       </joint>

File: sr_description/hand/xacro/finger/knuckle/knuckle.gazebo.xacro (robot description, xacro)
@@ -4,5 +4,4 @@
     <!-- prefix can be anything but usually is "r_" or  "l_" for right and left hands distinction -->
     <gazebo reference="${prefix}${link_prefix}knuckle">
-    <!-- knuckle is not highly exposed so bumper seems not useful
       <sensor type="contact" name="${prefix}${link_prefix}knuckle_contact">
         <always_on>1</always_on>
@@ -18,5 +17,5 @@
           <bumperTopicName>contacts/${prefix}${link_prefix}/knuckle</bumperTopicName>
         </plugin>
-      </sensor> -->
+      </sensor>
       <material>Gazebo/Grey</material>
     </gazebo>

File: sr_description/hand/xacro/full_hand.urdf.xacro (robot description, xacro)
@@ -1,6 +1,3 @@
-<robot xmlns:sensor="http://playerstage.sourceforge.net/gazebo/xmlschema/#sensor"
-xmlns:controller="http://playerstage.sourceforge.net/gazebo/xmlschema/#controller"
-xmlns:interface="http://playerstage.sourceforge.net/gazebo/xmlschema/#interface"
-xmlns:xacro="http://www.ros.org/wiki/xacro">
+<robot xmlns:sensor="http://playerstage.sourceforge.net/gazebo/xmlschema/#sensor" xmlns:controller="http://playerstage.sourceforge.net/gazebo/xmlschema/#controller" xmlns:interface="http://playerstage.sourceforge.net/gazebo/xmlschema/#interface" xmlns:xacro="http://www.ros.org/wiki/xacro">
   <xacro:include filename="$(find sr_description)/hand/xacro/forearm/forearm.urdf.xacro" />
   <xacro:include filename="$(find sr_description)/hand/xacro/wrist/wrist.urdf.xacro" />
@@ -8,6 +5,12 @@
   <xacro:include filename="$(find sr_description)/hand/xacro/finger/fingers.urdf.xacro" />
   <xacro:include filename="$(find sr_description)/hand/xacro/thumb/thumb.urdf.xacro" />
-  <!-- hand_type describes the hand type, hand_e, hand_e_plus, hand_m (muscle) -->
-  <!-- fingers describes which fingers are present, [th, ff, mf, rf, lf], default [1, 1, 1, 1, 1] -->
+  <!-- hand_type can be: hand_e, hand_e_plus, hand_m (muscle), hand_mt (muscletrans) -->
+  <!-- fingers: dict specifying available fingers, default: dict(th=1, ff=1, mf=1, rf=1, lf=1) -->
+  <!-- tip_sensors: dict specifying the fingertip (tactile) sensors per finger: std, none, bio, bt_sp, ubi, eli -->
+  <!-- mid_sensors: dict specifying the middle-phalange (tactile) sensors per finger: std, none, bio, ubi -->
+  <!-- prox_sensors: dict specifying the proximal (tactile) sensors per finger: std, none, ubi -->
+  <!-- palm_sensor: specifies the palm tactile sensor: std, none, ubi -->
+  <!-- reflect is either 1 (for right hand) or -1 (for left hand) -->
+  <!-- prefix can be anything but usually is "r_" or  "l_" for right and left hands distinction -->
   <!-- muscletrans (deprecated) is true for muscle transmission to be used, false to use motor transmission -->
   <!-- muscle (deprecated) is true for muscle hand or false for motor hand -->
@@ -16,16 +19,8 @@
   <!-- ubi (deprecated) is true for ubi finger or false for standard finger -->
   <!-- eli (deprecated) is true for ellipsoid fingertip or false for standard finger -->
-  <!-- tip_sensors vector that describes the sensor std, none, bio, bt_sp, ubi, eli -->
-  <!-- mid_sensors vector that describes the sensor std, none, bio, ubi -->
-  <!-- prox_sensors vector that describes the sensor std, none, ubi -->
-  <!-- palm_sensor describes the sensor std, none, ubi -->
-  <!-- reflect is either 1 (for right hand) or -1 (for left hand) -->
-  <!-- prefix can be anything but usually is "r_" or  "l_" for right and left hands distinction -->
   <!-- lf (deprecated) is true if we want a little finger, false otherwise -->
-  <xacro:macro name="shadowhand"
-  params="hand_type:='hand_e' reflect prefix cable_mesh:=False
-          fingers:=${[1,1,1,1,1]} tip_sensors:=${['std','std','std','std','std']} prox_sensors:=${['std','std','std','std','std']}
-          mid_sensors:=${['std','std','std','std','std']} palm_sensor:=std
-          muscletrans:=False muscle:=False lf:=True bio:=False bt_sp:=False ubi:=False eli:=False">
+  <xacro:macro name="shadowhand" params="hand_type:='hand_e' reflect prefix cable_mesh:=False fingers:=${[1,1,1,1,1]}
+          tip_sensors:=${5 * ['std']} mid_sensors:=${5 * ['std']} prox_sensors:=${5 * ['std']} palm_sensor:=std
+          muscletrans:=^|False muscle:=^|False lf:=^|True bio:=^|False bt_sp:=^|False ubi:=^|False eli:=^|False">
     <!-- handle deprecated parameters -->
     <xacro:include filename="$(find sr_description)/hand/xacro/backward_compat.urdf.xacro" />
@@ -47,7 +42,5 @@
     <!-- First Finger -->
     <xacro:if value="${fingers[1] == 1}">
-      <xacro:finger link_prefix="ff" joint_prefix="FF" tip_sensor="${tip_sensors[1]}"
-                    prox_sensor="${prox_sensors[1]}" mid_sensor="${mid_sensors[1]}"
-                    parent="${prefix}palm">
+      <xacro:finger link_prefix="ff" joint_prefix="FF" tip_sensor="${tip_sensors[1]}" prox_sensor="${prox_sensors[1]}" mid_sensor="${mid_sensors[1]}" parent="${prefix}palm">
         <origin xyz="${reflect*0.033} 0 0.095" rpy="0 0 0" />
         <axis xyz="0 ${-1*reflect} 0" />
@@ -56,7 +49,5 @@
     <!-- Middle Finger -->
     <xacro:if value="${fingers[2] == 1}">
-      <xacro:finger link_prefix="mf" joint_prefix="MF" tip_sensor="${tip_sensors[2]}"
-                    prox_sensor="${prox_sensors[2]}" mid_sensor="${mid_sensors[2]}"
-                    parent="${prefix}palm">
+      <xacro:finger link_prefix="mf" joint_prefix="MF" tip_sensor="${tip_sensors[2]}" prox_sensor="${prox_sensors[2]}" mid_sensor="${mid_sensors[2]}" parent="${prefix}palm">
         <origin xyz="${reflect*0.011} 0 0.099" rpy="0 0 0" />
         <axis xyz="0 ${-1*reflect} 0" />
@@ -65,7 +56,5 @@
     <!-- Ring Finger -->
     <xacro:if value="${fingers[3] == 1}">
-      <xacro:finger link_prefix="rf" joint_prefix="RF" tip_sensor="${tip_sensors[3]}"
-                    prox_sensor="${prox_sensors[3]}" mid_sensor="${mid_sensors[3]}"
-                    parent="${prefix}palm">
+      <xacro:finger link_prefix="rf" joint_prefix="RF" tip_sensor="${tip_sensors[3]}" prox_sensor="${prox_sensors[3]}" mid_sensor="${mid_sensors[3]}" parent="${prefix}palm">
         <origin xyz="${reflect*-0.011} 0 0.095" rpy="0 0 0" />
         <axis xyz="0 ${reflect} 0" />
@@ -73,8 +62,6 @@
     </xacro:if>
     <!-- Little Finger  -->
-    <xacro:if value="${fingers[4] == 1}">
-      <xacro:finger link_prefix="lf" joint_prefix="LF" tip_sensor="${tip_sensors[4]}"
-                    prox_sensor="${prox_sensors[4]}" mid_sensor="${mid_sensors[4]}"
-                    parent="${prefix}palm">
+    <xacro:if value="${fingers[4] == 1 and lf}">
+      <xacro:finger link_prefix="lf" joint_prefix="LF" tip_sensor="${tip_sensors[4]}" prox_sensor="${prox_sensors[4]}" mid_sensor="${mid_sensors[4]}" parent="${prefix}palm">
         <origin xyz="0 0 0.06579" rpy="0 0 0" />
         <axis xyz="0 ${reflect} 0" />
@@ -83,6 +70,5 @@
     <!-- Thumb  -->
     <xacro:if value="${fingers[0] == 1}">
-      <xacro:thumb is_lite="0" parent="${prefix}palm" tip_sensor="${tip_sensors[0]}"
-                   prox_sensor="${prox_sensors[0]}" mid_sensor="${mid_sensors[0]}" />
+      <xacro:thumb is_lite="0" parent="${prefix}palm" tip_sensor="${tip_sensors[0]}" prox_sensor="${prox_sensors[0]}" mid_sensor="${mid_sensors[0]}" />
     </xacro:if>
   </xacro:macro>

File: sr_description/hand/xacro/hand_lite.urdf.xacro (robot description, xacro)
@@ -8,6 +8,13 @@
   <xacro:include filename="$(find sr_description)/hand/xacro/finger/fingers.urdf.xacro" />
   <xacro:include filename="$(find sr_description)/hand/xacro/thumb/thumb.urdf.xacro" />
-  <!-- hand_type describes the hand type, hand_e, hand_e_plus, hand_m (muscle) -->
-  <!-- extra_lite (deprecated) describes if the hand is extra_lite -->
+  <!-- hand_type can be: hand_e, hand_e_plus, hand_m (muscle), hand_mt (muscletrans) -->
+  <!-- fingers: dict specifying available fingers, default: dict(th=1, ff=1, mf=1, rf=1, lf=1) -->
+  <!-- tip_sensors: dict specifying the fingertip (tactile) sensors per finger: std, none, bio, bt_sp, ubi, eli -->
+  <!-- mid_sensors: dict specifying the middle-phalange (tactile) sensors per finger: std, none, bio, ubi -->
+  <!-- prox_sensors: dict specifying the proximal (tactile) sensors per finger: std, none, ubi -->
+  <!-- palm_sensor: specifies the palm tactile sensor: std, none, ubi -->
+  <!-- reflect is either 1 (for right hand) or -1 (for left hand) -->
+  <!-- prefix can be anything but usually is "r_" or  "l_" for right and left hands distinction -->
+  <!-- extra_lite (deprecated) describes if the hand is extra_lite, i.e. without MF -->
   <!-- muscletrans (deprecated) is true for muscle transmission to be used, false to use motor transmission -->
   <!-- muscle (deprecated) is true for muscle hand or false for motor hand -->
@@ -16,19 +23,12 @@
   <!-- ubi (deprecated) is true for ubi finger or false for standard finger -->
   <!-- eli (deprecated) is true for ellipsoid fingertip or false for standard finger -->
-  <!-- tip_sensors vector that describes the sensor std, none, bio, bt_sp, ubi, eli -->
-  <!-- mid_sensors vector that describes the sensor std, none, bio, ubi -->
-  <!-- prox_sensors vector that describes the sensor std, none, ubi -->
-  <!-- palm_sensor describes the sensor none, bumper, ubi -->
-  <!-- reflect is either 1 (for right hand) or -1 (for left hand) -->
-  <!-- prefix can be anything but usually is "r_" or  "l_" for right and left hands distinction -->
   <xacro:macro name="shadowhand"
-  params="hand_type:='hand_e' reflect prefix cable_mesh:=False
-          fingers:=${[1,1,1,1]} tip_sensors:=${['std','std','std','std']} prox_sensors:=${['std','std','std','std']}
-          mid_sensors:=${['std','std','std','std']} palm_sensor:=std
-          muscletrans:=False muscle:=False lf:=True extra_lite:=False bio:=False bt_sp:=False ubi:=False eli:=False">
+  params="hand_type:='hand_e' reflect prefix cable_mesh:=False fingers:=${[1,1,1,1]}
+          tip_sensors:=${4 * ['std']} mid_sensors:=${4 * ['std']} prox_sensors:=${4 * ['std']} palm_sensor:=std
+          extra_lite:=^|False muscletrans:=^|False muscle:=^|False bio:=^|False bt_sp:=^|False ubi:=^|False eli:=^|False">
     <!-- handle deprecated parameters -->
     <xacro:include filename="$(find sr_description)/hand/xacro/backward_compat.urdf.xacro" />
     <xacro:if value="${extra_lite}">
-      <xacro:property name="fingers" value="${[1,0,1,1]}"/>
+      <xacro:property name="fingers" value="${[1,1,0,1]}" />
     </xacro:if>
     <!-- Forearm -->

File: sr_description/hand/xacro/thumb/thbase.gazebo.xacro (robot description, xacro)
@@ -4,5 +4,4 @@
     <!-- prefix can be anything but usually is "r_" or  "l_" for right and left hands distinction -->
     <gazebo reference="${prefix}thbase">
-      <!-- base is inside the proximal and not exposed so bumper seems useless
       <sensor type="contact" name="${prefix}thbase_contact">
         <always_on>1</always_on>
@@ -18,5 +17,5 @@
           <bumperTopicName>contacts/${prefix}th/base</bumperTopicName>
         </plugin>
-      </sensor> -->
+      </sensor>
       <selfCollide>false</selfCollide>
     </gazebo>

File: sr_description/hand/xacro/thumb/thhub.gazebo.xacro (robot description, xacro)
@@ -4,5 +4,4 @@
     <!-- prefix can be anything but usually is "r_" or  "l_" for right and left hands distinction -->
     <gazebo reference="${prefix}thhub">
-      <!-- hub is inside the proximal and not exposed so bumper seems useless
       <sensor type="contact" name="${prefix}thhub_contact">
         <always_on>1</always_on>
@@ -18,6 +17,6 @@
           <bumperTopicName>contacts/${prefix}th/hub</bumperTopicName>
         </plugin>
-      </sensor> -->
-      <selfCollide>false</selfCollide>
+      </sensor>
+      <selfCollide>true</selfCollide>
     </gazebo>
   </xacro:macro>

File: sr_description/hand/xacro/thumb/thmiddle.urdf.xacro (robot description, xacro)
@@ -63,5 +63,5 @@
       <parent link="${parent}" />
       <child link="${prefix}thmiddle" />
-      <xacro:if value="${bio}">
+      <xacro:if value="${'bio' in mid_sensor}">
         <origin xyz="0 0 0.01" rpy="0 0 0" />
         <!-- FIXME: z offset is too large -->

File: sr_description/hand/xacro/thumb/thumb.urdf.xacro (robot description, xacro)
@@ -14,4 +14,7 @@
   <xacro:macro name="thumb"
   params=" tip_sensor:=^|'std' mid_sensor:=^|'std' prox_sensor:=^|'std' reflect:=^ prefix:=^ parent is_lite">
+    <xacro:if value="${tip_sensor == 'bio'}">
+      <xacro:property name="mid_sensor" value="bio" />
+    </xacro:if>
     <!-- Base -->
     <xacro:thbase parent="${parent}" />

File: sr_description/robots/arm_and_sr_one_finger_motor.urdf.xacro (robot description, xacro)
@@ -19,5 +19,4 @@
     <dynamics damping="3.5" />
   </joint>
-  <xacro:shadowhand muscletrans="false" muscle="false" bio="false" bt_sp="false"
-  ubi="false" eli="false" reflect="1.0" prefix="rh_" />
+  <xacro:shadowhand reflect="1.0" prefix="rh_" />
 </robot>

File: sr_description/robots/bimanual_shadowhand_extra_lite.urdf.xacro (robot description, xacro)
@@ -11,5 +11,5 @@
     <origin xyz="0.0 0.0 0.0" rpy="0.0 0.0 0.0" />
   </joint>
-  <xacro:shadowhand hand_type="hand_e" fingers="${[1,0,1,1]}" reflect="1.0" prefix="rh_" />
+  <xacro:shadowhand hand_type="hand_e" fingers="${[1,1,0,1]}" reflect="1.0" prefix="rh_" />
   <joint name="right_hand_to_left_hand" type="fixed">
     <parent link="rh_forearm" />
@@ -17,4 +17,4 @@
     <origin xyz="$(arg arm_x_separation) 0.0 0.0" rpy="0.0 0.0 0.0" />
   </joint>
-  <xacro:shadowhand hand_type="hand_e" fingers="${[1,0,1,1]}" reflect="-1.0" prefix="lh_" />
+  <xacro:shadowhand hand_type="hand_e" fingers="${[1,1,0,1]}" reflect="-1.0" prefix="lh_" />
 </robot>

File: sr_description/robots/bimanual_shadowhand_lite_btsp.urdf.xacro (robot description, xacro)
@@ -11,5 +11,5 @@
     <origin xyz="0.0 0.0 0.0" rpy="0.0 0.0 0.0" />
   </joint>
-  <xacro:shadowhand hand_type="hand_e" tip_sensors="${['bt_sp','bt_sp','bt_sp','bt_sp','bt_sp']}" reflect="1.0" prefix="rh_" />
+  <xacro:shadowhand hand_type="hand_e" tip_sensors="${5 * ['bt_sp']}" reflect="1.0" prefix="rh_" />
   <joint name="right_hand_to_left_hand" type="fixed">
     <parent link="rh_forearm" />
@@ -17,4 +17,4 @@
     <origin xyz="$(arg arm_x_separation) 0.0 0.0" rpy="0.0 0.0 0.0" />
   </joint>
-  <xacro:shadowhand hand_type="hand_e" tip_sensors="${['bt_sp','bt_sp','bt_sp','bt_sp','bt_sp']}" reflect="-1.0" prefix="lh_" />
+  <xacro:shadowhand hand_type="hand_e" tip_sensors="${5 * ['bt_sp']}" reflect="-1.0" prefix="lh_" />
 </robot>

File: sr_description/robots/shadowhand_extra_lite.urdf.xacro (robot description, xacro)
@@ -14,4 +14,4 @@
     <origin xyz="0.0 0.0 0.0" rpy="0.0 0.0 0.0" />
   </joint>
-  <xacro:shadowhand hand_type="hand_e" fingers="${[1,0,1,1]}" reflect="1.0" prefix="rh_" />
+  <xacro:shadowhand hand_type="hand_e" fingers="${[1,1,0,1]}" reflect="1.0" prefix="rh_" />
 </robot>

File: sr_description/robots/shadowhand_left_extra_lite.urdf.xacro (robot description, xacro)
@@ -14,4 +14,4 @@
     <origin xyz="0.0 0.0 0.0" rpy="0.0 0.0 0.0" />
   </joint>
-  <xacro:shadowhand hand_type="hand_e" fingers="${[1,0,1,1]}" reflect="-1.0" prefix="lh_" />
+  <xacro:shadowhand hand_type="hand_e" fingers="${[1,1,0,1]}" reflect="-1.0" prefix="lh_" />
 </robot>

File: sr_description/robots/sr_one_finger_motor.urdf.xacro (robot description, xacro)
@@ -14,5 +14,4 @@
     <origin xyz="0.0 0.0 0.0" rpy="0.0 0.0 0.0" />
   </joint>
-  <xacro:shadowhand muscletrans="false" muscle="false" bio="false" bt_sp="false"
-  ubi="false" eli="false" reflect="1.0" prefix="rh_" />
+  <xacro:shadowhand reflect="1.0" prefix="rh_" />
 </robot>

File: sr_description/robots/sr_three_finger_edc_muscle_biotac.urdf.xacro (robot description, xacro)
@@ -14,4 +14,4 @@
     <origin xyz="0.0 0.0 0.0" rpy="0.0 0.0 0.0" />
   </joint>
-  <xacro:shadowhand hand_type="hand_m" fingers="${[1,1,1,0,0]}" tip_sensors="${['bio','bio','bio','std','std']}" reflect="1.0" prefix="rh_" />
+  <xacro:shadowhand hand_type="hand_mt" fingers="${[1,1,1,0,0]}" tip_sensors="${['bio','bio','bio','std','std']}" reflect="1.0" prefix="rh_" />
 </robot>
