Commit message: Passing params. Still failing in str

File: sr_description/robots/sr_hand_e.urdf.xacro (robot description, xacro)
@@ -9,9 +9,10 @@
     <xacro:arg name="hand_version" default="E3M5"/>
     <xacro:arg name="side" default="right"/>
-    <xacro:arg name="fingers" default="${[1,1,1,1,1]}"/>
-    <xacro:arg name="tip_sensors" default="${['pst','pst','pst','pst','pst']}"/>
-    <xacro:arg name="mid_sensors" default="${['none','none','none','none','none']}"/>
-    <xacro:arg name="prox_sensors" default="${['none','none','none','none','none']}"/>
+    <xacro:arg name="fingers" default="1,1,1,1,1"/>
+    <xacro:arg name="tip_sensors" default="'pst','bt_sp','pst','pst','pst'"/>
+    <xacro:arg name="mid_sensors" default="'none','none','none','none','none'"/>
+    <xacro:arg name="prox_sensors" default="'none','none','none','none','none'"/>
     <xacro:arg name="palm_sensor" default="none"/>
+    <xacro:property name="tip_sensors_p" default="${($(arg tip_sensors))}"/>
     <link name="world" />
     <joint name="rh_world_joint" type="fixed">
@@ -20,4 +21,5 @@
       <origin xyz="0.0 0.0 0.0" rpy="0.0 0.0 0.0" />
     </joint>
-    <xacro:sr_hand hand_version="$(arg hand_version)" side="$(arg side)" fingers="$(arg fingers)" tip_sensors="$(arg tip_sensors)" mid_sensors="$(arg mid_sensors)" prox_sensors="$(arg prox_sensors)" palm_sensor="$(arg palm_sensor)"/>
+    <!--xacro:sr_hand hand_version="$(arg hand_version)" side="$(arg side)" fingers="${($(arg fingers))}" tip_sensors="${($(arg tip_sensors))}" mid_sensors="${($(arg mid_sensors))}" prox_sensors="${($(arg prox_sensors))}" palm_sensor="${($(arg palm_sensor))}"/-->
+    <xacro:sr_hand hand_version="$(arg hand_version)" side="$(arg side)" fingers="${($(arg fingers))}" tip_sensors="${($(arg tip_sensors))}"/>
 </robot>
