Commit message: More simplifications
- Simpify one_finger_unit.urdf.xacro
  There is only one finger. No need to pass *_sensors. A single one is sufficient.
  Also, a fingers parameter doesn't make sense.

- Reduce number of xacro:if in fingers.urdf.xacro

- Plain string default parameters don't need to be quoted

File: sr_description/hand/xacro/finger/biotac/biotac.urdf.xacro (robot description, xacro)
@@ -12,5 +12,5 @@
   <!-- parent is the parent link for the joint -->
   <xacro:macro name="biotac_middle"
-  params="prefix:=^ link_prefix:=^ joint_prefix:=^ tip_sensor:=^|'std' mid_sensor:=^|standard parent">
+  params="prefix:=^ link_prefix:=^ joint_prefix:=^ tip_sensor:=^|std mid_sensor:=^|std parent">
     <link name="${prefix}${link_prefix}middle">
       <inertial>

File: sr_description/hand/xacro/finger/distal/distal.urdf.xacro (robot description, xacro)
@@ -14,5 +14,5 @@
   <!-- parent is the parent link for the joint -->
   <xacro:macro name="distal"
-  params="prefix:=^ link_prefix:=^ joint_prefix:=^ tip_sensor:=^|'std' parent">
+  params="prefix:=^ link_prefix:=^ joint_prefix:=^ tip_sensor:=^|std parent">
     <link name="${prefix}${link_prefix}distal">
       <inertial>

File: sr_description/hand/xacro/finger/fingers.urdf.xacro (robot description, xacro)
@@ -16,5 +16,5 @@
   <!-- parent is the parent link for the first joint -->
   <xacro:macro name="finger"
-  params="tip_sensor:=^|'std' mid_sensor:=^|'std' prox_sensor:=^|'std' reflect:=^ prefix:=^ link_prefix joint_prefix parent *origin *axis">
+  params="tip_sensor:=^|std mid_sensor:=^|std prox_sensor:=^|std reflect:=^ prefix:=^ link_prefix joint_prefix parent *origin *axis">
     <!-- Little finger special case -->
     <xacro:if value="${'lf' in link_prefix}">
@@ -34,16 +34,14 @@
     <!-- Proximal -->
     <xacro:proximal parent="${prefix}${link_prefix}knuckle"></xacro:proximal>
-    <!-- Biotac Middle -->
+    <!-- BioTac combines Middle + Distal -->
     <xacro:if value="${'bio' in tip_sensor}">
       <xacro:biotac_middle parent="${prefix}${link_prefix}proximal">
       </xacro:biotac_middle>
     </xacro:if>
-    <!-- Standard Middle -->
+    <!-- Non-BioTac -->
     <xacro:unless value="${'bio' in tip_sensor}">
+      <!-- Middle -->
       <xacro:middle parent="${prefix}${link_prefix}proximal"></xacro:middle>
-    </xacro:unless>
-    <!-- Distal  -->
-    <!-- only if finger is not biotac  -->
-    <xacro:unless value="${'bio' in tip_sensor}">
+      <!-- Distal  -->
       <xacro:distal parent="${prefix}${link_prefix}middle"></xacro:distal>
     </xacro:unless>

File: sr_description/hand/xacro/one_finger_unit.urdf.xacro (robot description, xacro)
@@ -20,7 +20,9 @@
   <!-- prefix can be anything but usually is "r_" or  "l_" for right and left hands distinction -->
   <xacro:macro name="shadowhand" params="hand_type:='hand_e' reflect prefix cable_mesh:=False
-          fingers:=${[1,1,1,1]} tip_sensors:=${['std','std','std','std']} prox_sensors:=${['std','std','std','std']}
-          mid_sensors:=${['std','std','std','std']} palm_sensor:=std
-          muscletrans:=False muscle:=False lf:=True extra_lite:=False bio:=False bt_sp:=False ubi:=False eli:=False">
+          tip_sensor:=std mid_sensor:=std prox_sensor:=std palm_sensor:=std
+          muscletrans:=False muscle:=False bio:=False bt_sp:=False ubi:=False eli:=False">
+    <xacro:property name="tip_sensors" value="${5 * [tip_sensor]}" />
+    <xacro:property name="mid_sensors" value="${5 * [mid_sensor]}" />
+    <xacro:property name="prox_sensors" value="${5 * [prox_sensor]}" />
     <xacro:include filename="$(find sr_description)/hand/xacro/backward_compat.urdf.xacro" />
     <!-- Forearm -->
@@ -57,12 +59,10 @@
     <!-- Middle Finger -->
     <!-- TODO: Check if offset is the same for muscle hand -->
-    <xacro:if value="${fingers[2] == 1}">
-      <xacro:finger link_prefix="mf" joint_prefix="MF" tip_sensor="${tip_sensors[2]}"
-                    prox_sensor="${prox_sensors[2]}" mid_sensor="${mid_sensors[2]}"
-                    parent="${prefix}palm">
-        <origin xyz="0.0 0 0.116" rpy="0 0 0" />
-        <axis xyz="0 ${-1*reflect} 0" />
-      </xacro:finger>
-    </xacro:if>
+    <xacro:finger link_prefix="mf" joint_prefix="MF" tip_sensor="${tip_sensors[2]}"
+                  prox_sensor="${prox_sensors[2]}" mid_sensor="${mid_sensors[2]}"
+                  parent="${prefix}palm">
+      <origin xyz="0.0 0 0.116" rpy="0 0 0" />
+      <axis xyz="0 ${-1*reflect} 0" />
+    </xacro:finger>
   </xacro:macro>
 </robot>

File: sr_description/hand/xacro/thumb/thumb.urdf.xacro (robot description, xacro)
@@ -13,5 +13,5 @@
   <!-- is_lite is this the lite hand, if so lock J3 -->
   <xacro:macro name="thumb"
-  params=" tip_sensor:=^|'std' mid_sensor:=^|'std' prox_sensor:=^|'std' reflect:=^ prefix:=^ parent is_lite">
+  params=" tip_sensor:=^|std mid_sensor:=^|std prox_sensor:=^|std reflect:=^ prefix:=^ parent is_lite">
     <xacro:if value="${tip_sensor == 'bio'}">
       <xacro:property name="mid_sensor" value="bio" />
